Commit message: temp

File: src/a_description/urdf/a.xacro (robot description, xacro)
@@ -1,9 +1,4 @@
 <?xml version="1.0" ?>
 <robot name="a" xmlns:xacro="http://www.ros.org/wiki/xacro">
-<link name="world"/>
-  <joint name="fixed_base" type="fixed">
-    <parent link="world"/>
-    <child link="base_link"/>
-  </joint>
 <xacro:include filename="$(find a_description)/urdf/materials.xacro" />
 <xacro:include filename="$(find a_description)/urdf/a.trans" />
@@ -11,15 +6,15 @@
 <link name="base_link">
   <inertial>
-    <origin xyz="5.228401932452191e-13 0.0 0.0015" rpy="0 0 0"/>
-    <mass value="0.00185"/>
-    <inertia ixx="0.0" iyy="0.0" izz="0.0" ixy="0.0" iyz="0.0" ixz="-0.0"/>
+    <origin xyz="-1.1580046200244058e-17 5.790023100122029e-18 0.024999999999999994" rpy="0 0 0"/>
+    <mass value="3.082687791334984"/>
+    <inertia ixx="0.002569" iyy="0.002569" izz="0.003853" ixy="-0.0" iyz="-0.0" ixz="-0.0"/>
   </inertial>
   <visual>
-      <origin xyz="0 0 0" rpy="0 0 0"/>
-      <geometry>
-        <mesh filename="package://a_description/meshes/base_link.stl" scale="0.001 0.001 0.001"/>
-      </geometry>
-      <material name="silver"/>
-    </visual>
+    <origin xyz="0 0 0" rpy="0 0 0"/>
+    <geometry>
+      <mesh filename="package://a_description/meshes/base_link.stl" scale="0.001 0.001 0.001"/>
+    </geometry>
+    <material name="silver"/>
+  </visual>
   <collision>
     <origin xyz="0 0 0" rpy="0 0 0"/>
@@ -149,5 +144,5 @@
   </collision>
 </link>
-<joint name="Revolute_18" type="continuous">
+<joint name="Revolute 18" type="continuous">
   <origin xyz="0.0 0.0 0.05" rpy="0 0 0"/>
   <parent link="base_link"/>
@@ -155,5 +150,5 @@
   <axis xyz="0.0 0.0 1.0"/>
 </joint>
-<joint name="Revolute_19" type="continuous">
+<joint name="Revolute 19" type="continuous">
   <origin xyz="0.075 -0.0 0.05" rpy="0 0 0"/>
   <parent link="link_1_1"/>
@@ -161,5 +156,5 @@
   <axis xyz="1.0 0.0 0.0"/>
 </joint>
-<joint name="Revolute_20" type="continuous">
+<joint name="Revolute 20" type="continuous">
   <origin xyz="0.05 0.0 0.075" rpy="0 0 0"/>
   <parent link="link_2_1"/>
@@ -167,5 +162,5 @@
   <axis xyz="0.0 0.0 1.0"/>
 </joint>
-<joint name="Revolute_21" type="continuous">
+<joint name="Revolute 21" type="continuous">
   <origin xyz="-0.075 0.0 0.05" rpy="0 0 0"/>
   <parent link="link_3_1"/>
@@ -173,5 +168,5 @@
   <axis xyz="-1.0 0.0 0.0"/>
 </joint>
-<joint name="Revolute_22" type="continuous">
+<joint name="Revolute 22" type="continuous">
   <origin xyz="-0.05 0.0 0.075" rpy="0 0 0"/>
   <parent link="link_4_1"/>
@@ -179,5 +174,5 @@
   <axis xyz="0.0 0.0 1.0"/>
 </joint>
-<joint name="Revolute_23" type="continuous">
+<joint name="Revolute 23" type="continuous">
   <origin xyz="0.075 0.0 0.05" rpy="0 0 0"/>
   <parent link="link_5_1"/>
